File: quadcopter.sch (EAGLE design)
At the start: 76 parts, among them J1 ISP, J3 POWER_JACKPTH_LOCK, M1 MOTOR_PADS, M2 MOTOR_PADS, M3 MOTOR_PADS, M4 MOTOR_PADS, Q1 CJ2302, Q2 CJ2302, Q3 CJ2302, Q4 CJ2302, U1 ATMEGA128RFA1, U2 LM1117, Y1 16MHz

Commit message: lab 4 complete
Parts:
- removed A1: ANTENNA2SMD5, SparkFun-RF:ANTENNA2SMD5
- removed C2: 0.1uF, quadparts_prebuilt:CAPACITOR-NP_SMD-2012-0805_CERAMIC-0.1UF
- removed C22, C23: 10uF, quadparts_prebuilt:CAPACITOR-NP_SMD-2012-0805_CERAMIC-10UF
- removed C8: 1uF, quadparts_prebuilt:CAPACITOR-NP_SMD-2012-0805_CERAMIC-1UF
- removed FID1, FID2: FIDUCIALUFIDUCIAL, SparkFun-Aesthetics:FIDUCIALUFIDUCIAL
- removed JP10, JP4: LOGO-SFENEW, SparkFun-Aesthetics:LOGO-SFENEW
- removed JP6: (no value), SparkFun-Connectors:M02JST-PTH-2
- removed JP7: (no value), SparkFun-Connectors:M021X02_NO_SILK
- removed JP8: (no value), SparkFun-Connectors:M023.5MM-NO_SILK
- removed LED1: RED, SparkFun-LED:LED0603
- removed LED2, LED3: GREEN, SparkFun-LED:LED0603
- removed M1, M2, M3, M4: MOTOR_PADS, Andranik-Lab4:MOTOR_PADS
- removed Q1, Q2, Q3, Q4: CJ2302, Seeed-Transistor-2016:SMD-MOSFET-N-CH-20V-2.1A-CJ2302(SOT-23)
- removed S2: (no value), SparkFun:SWITCH-SPST-SMD-A
- removed U1: ATMEGA128RFA1, SparkFun-DigitalIC:ATMEGA128RFA1
- removed U2: LM1117, SparkFun:V_REG_317SMD
- added BATT1: BATTERY-HUBSAN-W/HOLDER, quadparts_prebuilt:BATTERY-HUBSAN-W/HOLDER
- added D5, D6: green, quadparts_prebuilt:DIODE-LED_SMD-2012-0805-GREEN
- added J2: (no value), quadparts_ChengYuan:MALE_HEADER_2POS-2X1-0.1IN
- added R15: (no value), quadparts_prebuilt:RESISTOR_SMD-2012-0805
- added U$10, U$11, U$12, U$13: (no value), LEDs:RED_LED
- added U$14: ANTENNA2SMD5, quadparts_prebuilt:ANTENNA2SMD5
- added U$2, U$3, U$6, U$9: MOTOR_PADS, quadparts_prebuilt:MOTOR_PADS
- added U$4, U$5, U$7, U$8: (no value), quadparts_brandon:N_CHANNEL_MOSFET
- added U3: ATMEGA128RFA1, quadparts_prebuilt:ATMEGA128RFA1
- added V_REGULATOR: TPS73633-DBVT, quadparts_prebuilt:TPS73633-DBVT
- B1: value 748421245 -> BALUN0805; device SparkFun-RF:BALUN0805 -> quadparts_prebuilt:BALUN0805
- C3, C4: value JUMP -> 1uF; device quadparts_prebuilt:CAPACITOR-NP_SMD-2012-0805_CERAMIC -> quadparts_prebuilt:CAPACITOR-NP_SMD-2012-0805_CERAMIC-1UF
- J1: value ISP -> AVR_SPI_PRG_6NS; device SparkFun-Connectors:AVR_SPI_PRG_6NS -> quadparts_prebuilt:AVR_SPI_PRG_6NS
- J3: value POWER_JACKPTH_LOCK -> (none); device SparkFun-Connectors:POWER_JACKPTH_LOCK -> quadparts_brandon:BREAKOUT_HEADERTH-254X10
- JP9: value FTDI -> FTDI_BASICPTH; device SparkFun-Connectors:FTDI_BASICPTH -> quadparts_prebuilt:FTDI_BASICPTH
- R1: value 240 -> (none)
- R7, R8: value 1K -> (none)
- U$1: value OSHW-LOGOS -> (none); device SparkFun-Aesthetics:OSHW-LOGOS -> quadparts_brandon:NET_BRIDGE
- Y1: value 16MHz -> (none); device SparkFun-FreqCtrl:CRYSTAL5X3 -> quadparts_prebuilt:CRYSTAL5X3
Connections:
- removed net 3.3V: C20.1, C21.1, C23.1, C8.1, J1.2, JP9.4, R1.2, R11.2, R7.2, U1.DEVDD, U1.EVDD, U2.OUT
- removed net A0: U1.PF0(ADC0)
- removed net A1: U1.PF1(ADC1)
- removed net A2: U1.PF2(ADC2/DIG2)
- removed net A3: U1.PF3(ADC3/DIG4)
- removed net A4: U1.PF4(ADC4/TCK)
- removed net A5: U1.PF5(ADC5/TMS)
- removed net A6: U1.PF6(ADC6/TDO)
- removed net A7: U1.PF7(ADC7/TDI)
- removed net FB: R1.1, R8.2, U2.ADJ
- removed net N$15: C13.1, R2.1
- removed net N$16: C15.1, R6.1
- removed net N$17: C17.1, R13.1
- removed net N$21: C27.1, C28.1, IMU.VDD1, IMU.VDD2
- removed net N$22: C25.1, IMU.VDD_IO1
- removed net PE2: U1.PE2(XCK0/AIN0)
- removed net PE6: U1.PE6(T3/INT6)
- removed net PE7: U1.PE7(ICP3/INT7/CLKO)
- removed net RX0: JP9.3, U1.PE0(RXD0/PCINT8)
- removed net TX0: JP9.2, U1.PE1(TXD0)
- new net 3V: C20.1, C21.1, C4.1, J3.3V, R11.2, U3.DEVDD, U3.EVDD, V_REGULATOR.OUT
- new net BAT_GND: J3.BAT_GND, U$1.P$2
- net AREF: now also U3.AREF; no longer U1.AREF
- net AVDD: now also U3.AVDD; no longer U1.AVDD
- net DTR: now also JP9.6; no longer JP9.1
- net DVDD: now also U3.DVDD; no longer U1.DVDD
- net FILTERED: now also U$4.P$2, U$5.P$2, U$7.P$2, U$8.P$2; no longer Q1.G, Q2.G, Q3.G, Q4.G
- net FLYBACK: now also U$2.V-, U$3.V-, U$4.P$1, U$5.P$1, U$6.V-, U$7.P$1, U$8.P$1, U$9.V-; no longer M1.V-, M2.V-, M3.V-, M4.V-, Q1.D, Q2.D, Q3.D, Q4.D
- net GND: now also C3.2, C4.2, D5.C, D6.C, J2.1, JP9.1, U$1.P$1, U$10.PAS_POS, U$11.PAS_POS, U$12.PAS_POS, U$13.PAS_POS, U$4.P$3, U$5.P$3, U$7.P$3, U$8.P$3, U3.AVSS, U3.AVSS_RFN, U3.AVSS_RFP, U3.CLKI, U3.DVSS, U3.TST, V_REGULATOR.GND; no longer C2.2, C22.2, C23.2, C8.2, J3.GNDBREAK, JP6.1, JP7.1, JP8.1, JP9.6, LED1.C, LED2.C, LED3.C, Q1.S, Q2.S, Q3.S, Q4.S, R8.1, U1.AVSS, U1.AVSS_RFN, U1.AVSS_RFP, U1.CLKI, U1.DVSS, U1.PADDLE, U1.TST
- net MISO: now also U3.PB3(MISO/PDO/PCINT3); no longer U1.PB3(MISO/PDO/PCINT3)
- net MOSI: now also U3.PB2(MOSI/PDI/PCINT2); no longer U1.PB2(MOSI/PDI/PCINT2)
- net N$10: now also IMU.SDO_A/G; no longer B1.OUT1, C3.2
- net N$11: now also R15.2, U$13.PAS_NEG; no longer B1.OUT2, C4.2
- net N$13: now also D6.A; no longer LED2.A
- net N$2: now also R1.2, U$10.PAS_NEG; no longer LED1.A, R7.1
- net N$3: now also U3.XTAL1; no longer U1.XTAL1
- net N$4: now also U3.XTAL2; no longer U1.XTAL2
- net N$5: now also R7.2, U$11.PAS_NEG; no longer U1.PG4(TOSC1)
- net N$6: now also BATT1.N, J2.2; no longer U1.PG3(TOSC2)
- net N$8: now also D5.A; no longer LED3.A
- net N$9: now also R8.2, U$12.PAS_NEG; no longer J3.PWR, JP6.2, JP7.2, JP8.2, S2.P
- net PB4: now also U3.PB4(OC2A/PCINT4); no longer U1.PB4(OC2A/PCINT4)
- net PB5: now also J3.PB5, R15.1, U3.PB5(OC1A/PCINT5); no longer U1.PB5(OC1A/PCINT5)
- net PB6: now also U3.PB6(OC1B/PCINT6); no longer U1.PB6(OC1B/PCINT6)
- net PB7: now also U3.PB7(OC0A/OC1C/PCINT7); no longer U1.PB7(OC0A/OC1C/PCINT7)
- net PD4: now also U3.PD4(ICP1); no longer U1.PD4(ICP1)
- net PD5: now also U3.PD5(XCK1); no longer U1.PD5(XCK1)
- net PD6: now also U3.PD6(T1); no longer U1.PD6(T1)
- net PD7: now also U3.PD7(T0); no longer U1.PD7(T0)
- net PE3: now also C17.1, J3.PE3, R13.1, R7.1; no longer U1.PE3(OC3A/AIN1)
- net PE4: now also C15.1, J3.PE4, R6.1, R8.1; no longer U1.PE4(OC3B/INT4)
- net PE5: now also C13.1, J3.P5, R1.1, R2.1; no longer U1.PE5(OC3C/INT5)
- net PG0: now also U3.PG0(DIG3); no longer U1.PG0(DIG3)
- net PG1: now also U3.PG1(DIG1); no longer U1.PG1(DIG1)
- net PG2: now also U3.PG2(AMR); no longer U1.PG2(AMR)
- net PG5: now also U3.PG5(OC0B); no longer U1.PG5(OC0B)
- net RESET: now also U3.RSTN; no longer U1.RSTN
- net RFANT: now also U$14.SIGNAL; no longer A1.SIGNAL
- net RFN: now also B1.OUT2, U3.RFN; no longer C4.1, U1.RFN
- net RFP: now also B1.OUT1, U3.RFP; no longer C3.1, U1.RFP
- net RSTON: now also U3.RSTON; no longer U1.RSTON
- net RX1: now also JP9.4, U3.PD2(RXD1/INT2); no longer U1.PD2(RXD1/INT2)
- net SCK: now also U3.PB1(SCK/PCINT1); no longer U1.PB1(SCK/PCINT1)
- net SCL: now also IMU.SCL/SPC, J3.SCL, U3.PD0(SCL/INT0); no longer U1.PD0(SCL/INT0)
- net SDA: now also IMU.SDA/SDI/SDO, J3.SDA, U3.PD1(SDA/INT1); no longer U1.PD1(SDA/INT1)
- net SSN: now also U3.PB0(SSN/PCINT0); no longer U1.PB0(SSN/PCINT0)
- net TX1: now also JP9.5, U3.PD3(TXD1/INT3); no longer U1.PD3(TXD1/INT3)
- net VCC: now also BATT1.P, C25.1, C27.1, C28.1, C3.1, IMU.VDD1, IMU.VDD2, IMU.VDDIO2, IMU.VDD_IO1, J3.VBAT, U$2.V+, U$3.V+, U$6.V+, U$9.V+, V_REGULATOR.IN; no longer C2.1, C22.1, M1.V+, M2.V+, M3.V+, M4.V+, S2.O, U2.IN
Other:
- note removed: "800mA"
- note removed: "ADJ - 3.3V"
- note removed: "Jim Lindblom"
- note removed: "v23"
- moved on the sheet: C10, C11, C13, C14, C15, C16, C17, C20, C21, C3, C4, C6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

Commit message: finished lab 7
Parts:
- removed C25: 100nF, quadparts_prebuilt:CAPACITOR-NP_SMD-2012-0805_CERAMIC
- added C2: 220nF, quadparts_prebuilt:CAPACITOR-NP_SMD-2012-0805_CERAMIC
- added R16, R17, R18, R19, R20, R21: 10K, quadparts_prebuilt:RESISTOR_SMD-2012-0805-10K
- C10, C13, C15, C17: value 1uF -> 0.1uF
- C27: value 100nF -> 10nF
- R1, R15, R7, R8: value (none) -> 330
- U$10, U$11, U$12, U$13: value (none) -> RED
- U$15: value (none) -> LSM9DS1TR_9_AXIS_IMU
- renumbered IMU to U$15
Connections:
- removed net DTR: C1.1, JP9.6
- removed net FILTERED: R12.2, R13.2, R14.2, R2.2, R3.2, R4.2, R5.2, R6.2, U$4.P$2, U$5.P$2, U$7.P$2, U$8.P$2
- removed net FLYBACK: D1.A, D2.A, D3.A, D4.A, U$2.V-, U$3.V-, U$4.P$1, U$5.P$1, U$6.V-, U$7.P$1, U$8.P$1, U$9.V-
- removed net N$1: JPADDED.3
- removed net N$12: JPADDED.2
- new net FILTEREDNE: R12.2, R6.2, U$8.G
- new net FILTEREDNW: R3.2, R4.2, U$4.G
- new net FILTEREDSE: R13.2, R14.2, U$7.G
- new net FILTEREDSW: R2.2, R5.2, U$5.G
- new net FLYBACKNE: D3.A, U$6.V-, U$8.D
- new net FLYBACKNW: D2.A, U$2.V-, U$4.D
- new net FLYBACKSE: D4.A, U$7.D, U$9.V-
- new net FLYBACKSW: D1.A, U$3.V-, U$5.D
- new net N$15: R19.2, U$15.SDO_M
- new net N$16: R20.2, U$15.CS_A/G
- new net N$17: R21.2, U$15.CS_M
- new net N$21: C1.1, JP9.1
- new net RX0: JP9.2, U3.PE0(RXD0/PCINT8)
- new net TX0: JP9.3, U3.PE1(TXD0)
- net GND: now also BATT1.N, C2.2, JP9.6, U$4.S, U$5.S, U$7.S, U$8.S; no longer C25.2, J2.1, JP9.1, U$4.P$3, U$5.P$3, U$7.P$3, U$8.P$3
- net N$10: now also R18.2
- net N$6: now also BATT1.P, J2.1; no longer BATT1.N, J2.2
- net RX1: now also JPADDED.2; no longer JP9.4
- net SCL: now also R16.2
- net SDA: now also R17.2
- net TX1: now also JPADDED.3; no longer JP9.5
- net VCC: now also C2.1, J2.2, R16.1, R17.1, R18.1, R19.1, R20.1, R21.1, V_REGULATOR.EN; no longer BATT1.P, C25.1
Other:
- moved on the sheet: BATT1, C1, J2

Commit message: made changes to schematic/board per the comments the prof made
Parts:
- removed R20, R21: 10K, quadparts_prebuilt:RESISTOR_SMD-2012-0805-10K
- C24: value 10nF -> 10uF
Connections:
- net BAT_GND: now also C11.-, C14.-, C16.-, C2.2, C27.2, C28.2, C3.2, C6.-
- net GND: no longer C11.-, C14.-, C16.-, C2.2, C27.2, C28.2, C3.2, C6.-
- net N$16: now also R17.2, U$15.SCL/SPC; no longer R20.2, U$15.CS_A/G
- net N$17: now also R16.2, U$15.SDA/SDI/SDO; no longer R21.2, U$15.CS_M
- net PE3: now also U3.PE3(OC3A/AIN1)
- net PE4: now also U3.PE4(OC3B/INT4)
- net PE5: now also U3.PE5(OC3C/INT5)
- net SCL: no longer R16.2, U$15.SCL/SPC
- net SDA: no longer R17.2, U$15.SDA/SDI/SDO
- net VCC: now also U$15.CS_A/G, U$15.CS_M; no longer R20.1, R21.1
Other:
- moved on the sheet: R16, R17

Commit message: schematic changes for prof
Parts:
- removed C24: 10uF, quadparts_prebuilt:CAPACITOR-NP_SMD-2012-0805_CERAMIC
- removed C26: 100nF, quadparts_prebuilt:CAPACITOR-NP_SMD-2012-0805_CERAMIC
- added C22: 10uF, quadparts_prebuilt:CAPACITOR-NP_SMD-2012-0805_CERAMIC-10UF
- added C8: 0.1uF, quadparts_prebuilt:CAPACITOR-NP_SMD-2012-0805_CERAMIC-0.1UF
Connections:
- removed net N$19: C26.1
- net BAT_GND: now also U$4.S, U$5.S, U$7.S, U$8.S; no longer C2.2, C27.2, C28.2
- net GND: now also C2.2, C22.2, C27.2, C28.2, C8.1; no longer C24.2, U$4.S, U$5.S, U$7.S, U$8.S
- net N$18: now also C8.2; no longer C26.2
- net N$20: now also C22.1; no longer C24.1
- net RX0: now also JP9.3; no longer JP9.2
- net RX1: now also JPADDED.3; no longer JPADDED.2
- net TX0: now also JP9.2; no longer JP9.3
- net TX1: now also JPADDED.2; no longer JPADDED.3

Commit message: more changes made to board/schematic
Parts:
- removed R19: 10K, quadparts_prebuilt:RESISTOR_SMD-2012-0805-10K
Connections:
- net N$21 renamed DTR
- removed net N$15: R19.2, U$15.SDO_M
- removed net N$16: R17.2, U$15.SCL/SPC
- removed net N$17: R16.2, U$15.SDA/SDI/SDO
- net 3V: now also C2.1, C27.1, C28.1, R16.1, R17.1, R18.1, U$15.CS_A/G, U$15.CS_M, U$15.DEN_A/G, U$15.SDO_M, U$15.VDD1, U$15.VDD2, U$15.VDDIO2, U$15.VDD_IO1
- net SCL: now also R17.2, U$15.SCL/SPC
- net SDA: now also R16.2, U$15.SDA/SDI/SDO
- net VCC: no longer C2.1, C27.1, C28.1, R16.1, R17.1, R18.1, R19.1, U$15.CS_A/G, U$15.CS_M, U$15.VDD1, U$15.VDD2, U$15.VDDIO2, U$15.VDD_IO1

Commit message: schematic and board no longer inconsistent
Connections:
- net DTR renamed N$21
- removed net N$14: C10.1, R3.1
- net PB5: now also C10.1, R3.1
Changed lines of the file:
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@@
 <instance part="C22" gate="G$1" x="152.4" y="337.82" rot="R90"/>
 <instance part="GND39" gate="1" x="58.42" y="332.74"/>
-<instance part="P+1" gate="3V" x="96.52" y="378.46"/>
-<instance part="P+2" gate="3V" x="78.74" y="320.04"/>
-<instance part="P+4" gate="3V" x="60.96" y="284.48" rot="R90"/>
-<instance part="P+9" gate="3V" x="40.64" y="193.04" rot="R180"/>
-<instance part="P+10" gate="3V" x="149.86" y="220.98" rot="R180"/>
+<instance part="P+1" gate="3V" x="149.86" y="220.98" rot="R180"/>
+<instance part="P+2" gate="3V" x="40.64" y="193.04" rot="R180"/>
+<instance part="P+4" gate="3V" x="63.5" y="284.48" rot="R90"/>
+<instance part="P+9" gate="3V" x="78.74" y="320.04"/>
+<instance part="P+10" gate="3V" x="96.52" y="378.46"/>
 </instances>
 <busses>
@@
 <pinref part="GND30" gate="1" pin="GND"/>
 <wire x1="-81.28" y1="119.38" x2="-88.9" y2="119.38" width="0.1524" layer="91"/>
+<pinref part="BATT1" gate="G$1" pin="N"/>
 <wire x1="-88.9" y1="119.38" x2="-88.9" y2="116.84" width="0.1524" layer="91"/>
-<pinref part="BATT1" gate="G$1" pin="N"/>
 <wire x1="-91.44" y1="127" x2="-91.44" y2="119.38" width="0.1524" layer="91"/>
 <wire x1="-91.44" y1="119.38" x2="-88.9" y2="119.38" width="0.1524" layer="91"/>
+<junction x="-88.9" y="119.38"/>
 </segment>
 <segment>
@@
 <pinref part="R16" gate="G$1" pin="2"/>
 <wire x1="68.58" y1="271.78" x2="60.96" y2="271.78" width="0.1524" layer="91"/>
+<label x="63.5" y="276.86" size="1.778" layer="95" xref="yes"/>
 </segment>
 </net>
@@
 <pinref part="R17" gate="G$1" pin="2"/>
 <wire x1="68.58" y1="294.64" x2="60.96" y2="294.64" width="0.1524" layer="91"/>
+<label x="63.5" y="297.18" size="1.778" layer="95" xref="yes"/>
 </segment>
 </net>
@@
 </segment>
 <segment>
-<wire x1="-134.62" y1="210.82" x2="-139.7" y2="210.82" width="0.1524" layer="91"/>
-<label x="-139.7" y="210.82" size="1.778" layer="95" rot="R180" xref="yes"/>
-</segment>
-<segment>
 <pinref part="J3" gate="G$1" pin="PB5"/>
 <wire x1="215.9" y1="147.32" x2="226.06" y2="147.32" width="0.1524" layer="91"/>
@@
 <wire x1="132.08" y1="7.62" x2="124.46" y2="7.62" width="0.1524" layer="91"/>
 <label x="124.46" y="7.62" size="1.778" layer="95" rot="R180" xref="yes"/>
+</segment>
+<segment>
+<wire x1="-134.62" y1="210.82" x2="-143.002" y2="210.82" width="0.1524" layer="91"/>
+<label x="-143.002" y="210.82" size="1.778" layer="95" rot="R180" xref="yes"/>
+<pinref part="C10" gate="G$1" pin="1"/>
+<pinref part="R3" gate="G$1" pin="1"/>
+<wire x1="-124.46" y1="205.74" x2="-134.62" y2="205.74" width="0.1524" layer="91"/>
+<wire x1="-134.62" y1="205.74" x2="-134.62" y2="210.82" width="0.1524" layer="91"/>
+<junction x="-134.62" y="210.82"/>
 </segment>
 </net>
@@
 <wire x1="-58.42" y1="127" x2="-45.72" y2="127" width="0.1524" layer="91"/>
 <label x="-45.72" y="132.08" size="1.778" layer="95" rot="R90" xref="yes"/>
+<junction x="-45.72" y="127"/>
+<junction x="-38.1" y="127"/>
 </segment>
 <segment>
@@
 <pinref part="U$8" gate="G$1" pin="D"/>
 <wire x1="322.58" y1="223.52" x2="342.9" y2="223.52" width="0.1524" layer="91"/>
-</segment>
-</net>
-<net name="N$14" class="2">
-<segment>
-<pinref part="C10" gate="G$1" pin="1"/>
-<pinref part="R3" gate="G$1" pin="1"/>
-<wire x1="-124.46" y1="205.74" x2="-134.62" y2="205.74" width="0.1524" layer="91"/>
-<wire x1="-134.62" y1="205.74" x2="-134.62" y2="210.82" width="0.1524" layer="91"/>
+<junction x="322.58" y="224.79"/>
+<junction x="322.58" y="238.76"/>
 </segment>
 </net>
@@
 <wire x1="5.08" y1="132.08" x2="15.24" y2="132.08" width="0.1524" layer="91"/>
 <pinref part="P+3" gate="3V" pin="3V"/>
+<junction x="5.08" y="132.08"/>
 </segment>
 <segment>
@@
 </segment>
 <segment>
-<wire x1="106.68" y1="312.42" x2="106.68" y2="320.04" width="0.1524" layer="91"/>
-<wire x1="106.68" y1="320.04" x2="114.3" y2="320.04" width="0.1524" layer="91"/>
-<wire x1="114.3" y1="312.42" x2="114.3" y2="320.04" width="0.1524" layer="91"/>
-<wire x1="114.3" y1="320.04" x2="114.3" y2="368.3" width="0.1524" layer="91"/>
-<junction x="114.3" y="320.04"/>
-<wire x1="114.3" y1="368.3" x2="96.52" y2="368.3" width="0.1524" layer="91"/>
-<wire x1="96.52" y1="368.3" x2="96.52" y2="363.22" width="0.1524" layer="91"/>
-<wire x1="96.52" y1="363.22" x2="88.9" y2="363.22" width="0.1524" layer="91"/>
-<wire x1="88.9" y1="363.22" x2="81.28" y2="363.22" width="0.1524" layer="91"/>
-<wire x1="96.52" y1="363.22" x2="96.52" y2="358.14" width="0.1524" layer="91"/>
-<junction x="96.52" y="363.22"/>
-<pinref part="C28" gate="G$1" pin="1"/>
-<pinref part="C27" gate="G$1" pin="1"/>
-<wire x1="81.28" y1="363.22" x2="81.28" y2="360.68" width="0.1524" layer="91"/>
-<wire x1="96.52" y1="368.3" x2="96.52" y2="375.92" width="0.1524" layer="91"/>
-<junction x="96.52" y="368.3"/>
-<wire x1="88.9" y1="363.22" x2="88.9" y2="358.14" width="0.1524" layer="91"/>
-<pinref part="C2" gate="G$1" pin="1"/>
-<pinref part="U$15" gate="G$1" pin="VDD2"/>
-<pinref part="U$15" gate="G$1" pin="VDD1"/>
+<pinref part="U$15" gate="G$1" pin="DEN_A/G"/>
+<wire x1="149.86" y1="223.52" x2="149.86" y2="226.06" width="0.1524" layer="91"/>
 <pinref part="P+1" gate="3V" pin="3V"/>
-</segment>
-<segment>
-<wire x1="78.74" y1="312.42" x2="78.74" y2="317.5" width="0.1524" layer="91"/>
-<pinref part="U$15" gate="G$1" pin="VDD_IO1"/>
-<pinref part="P+2" gate="3V" pin="3V"/>
-</segment>
-<segment>
-<wire x1="68.58" y1="284.48" x2="63.5" y2="284.48" width="0.1524" layer="91"/>
-<pinref part="U$15" gate="G$1" pin="VDDIO2"/>
-<pinref part="P+4" gate="3V" pin="3V"/>
 </segment>
 <segment>
@@
 <pinref part="U$15" gate="G$1" pin="SDO_M"/>
 <wire x1="78.74" y1="226.06" x2="78.74" y2="203.2" width="0.1524" layer="91"/>
+<pinref part="P+2" gate="3V" pin="3V"/>
+</segment>
+<segment>
+<wire x1="68.58" y1="284.48" x2="66.04" y2="284.48" width="0.1524" layer="91"/>
+<pinref part="U$15" gate="G$1" pin="VDDIO2"/>
+<pinref part="P+4" gate="3V" pin="3V"/>
+</segment>
+<segment>
+<wire x1="78.74" y1="312.42" x2="78.74" y2="317.5" width="0.1524" layer="91"/>
+<pinref part="U$15" gate="G$1" pin="VDD_IO1"/>
 <pinref part="P+9" gate="3V" pin="3V"/>
 </segment>
 <segment>
-<pinref part="U$15" gate="G$1" pin="DEN_A/G"/>
+<wire x1="106.68" y1="312.42" x2="106.68" y2="320.04" width="0.1524" layer="91"/>
+<wire x1="106.68" y1="320.04" x2="114.3" y2="320.04" width="0.1524" layer="91"/>
+<wire x1="114.3" y1="312.42" x2="114.3" y2="320.04" width="0.1524" layer="91"/>
+<wire x1="114.3" y1="320.04" x2="114.3" y2="368.3" width="0.1524" layer="91"/>
+<junction x="114.3" y="320.04"/>
+<wire x1="114.3" y1="368.3" x2="96.52" y2="368.3" width="0.1524" layer="91"/>
+<wire x1="96.52" y1="368.3" x2="96.52" y2="363.22" width="0.1524" layer="91"/>
+<wire x1="96.52" y1="363.22" x2="88.9" y2="363.22" width="0.1524" layer="91"/>
+<wire x1="88.9" y1="363.22" x2="81.28" y2="363.22" width="0.1524" layer="91"/>
+<wire x1="96.52" y1="363.22" x2="96.52" y2="358.14" width="0.1524" layer="91"/>
+<junction x="96.52" y="363.22"/>
+<pinref part="C28" gate="G$1" pin="1"/>
+<pinref part="C27" gate="G$1" pin="1"/>
+<wire x1="81.28" y1="363.22" x2="81.28" y2="360.68" width="0.1524" layer="91"/>
+<wire x1="96.52" y1="368.3" x2="96.52" y2="375.92" width="0.1524" layer="91"/>
+<junction x="96.52" y="368.3"/>
+<wire x1="88.9" y1="363.22" x2="88.9" y2="358.14" width="0.1524" layer="91"/>
+<pinref part="C2" gate="G$1" pin="1"/>
+<pinref part="U$15" gate="G$1" pin="VDD2"/>
+<pinref part="U$15" gate="G$1" pin="VDD1"/>
+<junction x="88.9" y="363.22"/>
+<junction x="81.28" y="363.22"/>
 <pinref part="P+10" gate="3V" pin="3V"/>
-<wire x1="149.86" y1="223.52" x2="149.86" y2="226.06" width="0.1524" layer="91"/>
 </segment>
 </net>
@@
 </segment>
 </net>
-<net name="DTR" class="0">
+<net name="N$21" class="0">
 <segment>
 <pinref part="JP9" gate="G$1" pin="1"/>
@@
 <pinref part="U$4" gate="G$1" pin="D"/>
 <wire x1="-109.22" y1="218.44" x2="-88.9" y2="218.44" width="0.1524" layer="91"/>
+<junction x="-109.22" y="219.71"/>
 </segment>
 </net>
@@
 <wire x1="-101.6" y1="-25.4" x2="-78.74" y2="-25.4" width="0.1524" layer="91"/>
 <wire x1="-78.74" y1="-25.4" x2="-78.74" y2="-27.94" width="0.1524" layer="91"/>
+<junction x="-101.6" y="-25.4"/>
+<junction x="-101.6" y="-12.7"/>
 </segment>
 </net>
@@
 <pinref part="U$7" gate="G$1" pin="D"/>
 <wire x1="309.88" y1="-33.02" x2="330.2" y2="-33.02" width="0.1524" layer="91"/>
-</segment>
-</net>
+<junction x="309.88" y="-31.75"/>
+<junction x="309.88" y="-17.78"/>
+</segment>
+</net>
