File: quadcopter.sch (EAGLE design)
At the start: 73 parts, among them J1 AVR_SPI_PRG_6NS, U3 ATMEGA128RFA1

Commit message: made changes to pour
need to change RED LED to be more like data sheet
Connections:
- net FILTEREDNE: now also C15.1
- net FILTEREDNW: now also C10.1
- net FILTEREDSE: now also C17.1
- net FILTEREDSW: now also C13.1
- net PB5: no longer C10.1
- net PE3: no longer C17.1
- net PE4: no longer C15.1
- net PE5: no longer C13.1
Other:
- moved on the sheet: R13, R2, R3, R6
Changed lines of the file:
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@@
 <instance part="C6" gate="G$1" x="-137.16" y="233.68"/>
 <instance part="C10" gate="G$1" x="-124.46" y="203.2"/>
-<instance part="R3" gate="G$1" x="-129.54" y="210.82"/>
+<instance part="R3" gate="G$1" x="-137.16" y="210.82"/>
 <instance part="R4" gate="G$1" x="-114.3" y="198.12" rot="R90"/>
 <instance part="D1" gate="G$1" x="-93.98" y="-12.7" rot="R90"/>
 <instance part="C11" gate="G$1" x="-129.54" y="-12.7"/>
 <instance part="C13" gate="G$1" x="-116.84" y="-43.18"/>
-<instance part="R2" gate="G$1" x="-121.92" y="-35.56"/>
+<instance part="R2" gate="G$1" x="-132.08" y="-35.56"/>
 <instance part="R5" gate="G$1" x="-106.68" y="-48.26" rot="R90"/>
 <instance part="GND29" gate="1" x="-129.54" y="-55.88"/>
@@
 <instance part="C14" gate="G$1" x="294.64" y="238.76"/>
 <instance part="C15" gate="G$1" x="307.34" y="208.28"/>
-<instance part="R6" gate="G$1" x="302.26" y="215.9"/>
+<instance part="R6" gate="G$1" x="292.1" y="215.9"/>
 <instance part="R12" gate="G$1" x="317.5" y="203.2" rot="R90"/>
 <instance part="GND33" gate="1" x="294.64" y="195.58"/>
@@
 <instance part="C16" gate="G$1" x="281.94" y="-17.78"/>
 <instance part="C17" gate="G$1" x="294.64" y="-48.26"/>
-<instance part="R13" gate="G$1" x="289.56" y="-40.64"/>
+<instance part="R13" gate="G$1" x="281.94" y="-40.64"/>
 <instance part="R14" gate="G$1" x="304.8" y="-53.34" rot="R90"/>
 <instance part="GND35" gate="1" x="281.94" y="-60.96"/>
@@
 <net name="PE5" class="2">
 <segment>
-<pinref part="C13" gate="G$1" pin="1"/>
-<pinref part="R2" gate="G$1" pin="1"/>
-<wire x1="-116.84" y1="-40.64" x2="-127" y2="-40.64" width="0.1524" layer="91"/>
-<wire x1="-127" y1="-40.64" x2="-127" y2="-35.56" width="0.1524" layer="91"/>
-<wire x1="-127" y1="-35.56" x2="-134.62" y2="-35.56" width="0.1524" layer="91"/>
-<junction x="-127" y="-35.56"/>
-<label x="-134.62" y="-35.56" size="1.778" layer="95" rot="R180" xref="yes"/>
-</segment>
-<segment>
 <pinref part="J3" gate="G$1" pin="P5"/>
 <wire x1="215.9" y1="144.78" x2="233.68" y2="144.78" width="0.1524" layer="91"/>
@@
 <label x="30.48" y="38.1" size="1.778" layer="95" rot="R180" xref="yes"/>
 </segment>
+<segment>
+<pinref part="R2" gate="G$1" pin="1"/>
+<wire x1="-137.16" y1="-35.56" x2="-142.24" y2="-35.56" width="0.1524" layer="91"/>
+<label x="-142.24" y="-35.56" size="1.778" layer="95" rot="R180" xref="yes"/>
+</segment>
 </net>
 <net name="PE4" class="2">
-<segment>
-<pinref part="C15" gate="G$1" pin="1"/>
-<pinref part="R6" gate="G$1" pin="1"/>
-<wire x1="307.34" y1="210.82" x2="297.18" y2="210.82" width="0.1524" layer="91"/>
-<wire x1="297.18" y1="210.82" x2="297.18" y2="215.9" width="0.1524" layer="91"/>
-<wire x1="297.18" y1="215.9" x2="289.56" y2="215.9" width="0.1524" layer="91"/>
-<junction x="297.18" y="215.9"/>
-<label x="289.56" y="215.9" size="1.778" layer="95" rot="R180" xref="yes"/>
-</segment>
 <segment>
 <pinref part="J3" gate="G$1" pin="PE4"/>
@@
 <label x="30.48" y="40.64" size="1.778" layer="95" rot="R180" xref="yes"/>
 </segment>
+<segment>
+<pinref part="R6" gate="G$1" pin="1"/>
+<wire x1="287.02" y1="215.9" x2="281.94" y2="215.9" width="0.1524" layer="91"/>
+<label x="281.94" y="215.9" size="1.778" layer="95" rot="R180" xref="yes"/>
+</segment>
 </net>
 <net name="PE3" class="2">
 <segment>
-<pinref part="C17" gate="G$1" pin="1"/>
 <pinref part="R13" gate="G$1" pin="1"/>
-<wire x1="294.64" y1="-45.72" x2="284.48" y2="-45.72" width="0.1524" layer="91"/>
-<wire x1="284.48" y1="-45.72" x2="284.48" y2="-40.64" width="0.1524" layer="91"/>
-<wire x1="284.48" y1="-40.64" x2="276.86" y2="-40.64" width="0.1524" layer="91"/>
-<junction x="284.48" y="-40.64"/>
-<label x="276.86" y="-40.64" size="1.778" layer="95" rot="R180" xref="yes"/>
+<wire x1="276.86" y1="-40.64" x2="269.24" y2="-40.64" width="0.1524" layer="91"/>
+<label x="269.24" y="-40.64" size="1.778" layer="95" rot="R180" xref="yes"/>
 </segment>
 <segment>
@@
 </segment>
 <segment>
-<wire x1="-134.62" y1="210.82" x2="-143.002" y2="210.82" width="0.1524" layer="91"/>
-<label x="-143.002" y="210.82" size="1.778" layer="95" rot="R180" xref="yes"/>
-<pinref part="C10" gate="G$1" pin="1"/>
+<wire x1="-142.24" y1="210.82" x2="-148.082" y2="210.82" width="0.1524" layer="91"/>
+<label x="-148.082" y="210.82" size="1.778" layer="95" rot="R180" xref="yes"/>
 <pinref part="R3" gate="G$1" pin="1"/>
-<wire x1="-124.46" y1="205.74" x2="-134.62" y2="205.74" width="0.1524" layer="91"/>
-<wire x1="-134.62" y1="205.74" x2="-134.62" y2="210.82" width="0.1524" layer="91"/>
-<junction x="-134.62" y="210.82"/>
 </segment>
 </net>
@@
 <pinref part="R10" gate="G$1" pin="1"/>
 <pinref part="D6" gate="G$1" pin="A"/>
-</segment>
-</net>
-<net name="FILTEREDNE" class="2">
-<segment>
-<label x="295.91" y="220.98" size="1.778" layer="95" rot="R180" xref="yes"/>
-<pinref part="R6" gate="G$1" pin="2"/>
-<wire x1="312.42" y1="220.98" x2="295.91" y2="220.98" width="0.1524" layer="91"/>
-<wire x1="307.34" y1="215.9" x2="312.42" y2="215.9" width="0.1524" layer="91"/>
-<wire x1="312.42" y1="215.9" x2="317.5" y2="215.9" width="0.1524" layer="91"/>
-<wire x1="317.5" y1="215.9" x2="317.5" y2="210.82" width="0.1524" layer="91"/>
-<wire x1="312.42" y1="208.28" x2="312.42" y2="215.9" width="0.1524" layer="91"/>
-<junction x="312.42" y="215.9"/>
-<wire x1="312.42" y1="220.98" x2="312.42" y2="215.9" width="0.1524" layer="91"/>
-<pinref part="R12" gate="G$1" pin="2"/>
-<wire x1="312.42" y1="208.28" x2="317.5" y2="208.28" width="0.1524" layer="91"/>
-<wire x1="317.5" y1="210.82" x2="325.12" y2="210.82" width="0.1524" layer="91"/>
-<pinref part="U$8" gate="G$1" pin="G"/>
 </segment>
 </net>
@@
 <pinref part="R3" gate="G$1" pin="2"/>
 <wire x1="-119.38" y1="215.9" x2="-135.89" y2="215.9" width="0.1524" layer="91"/>
+<wire x1="-132.08" y1="210.82" x2="-124.46" y2="210.82" width="0.1524" layer="91"/>
 <wire x1="-124.46" y1="210.82" x2="-119.38" y2="210.82" width="0.1524" layer="91"/>
 <wire x1="-119.38" y1="210.82" x2="-114.3" y2="210.82" width="0.1524" layer="91"/>
@@
 <wire x1="-114.3" y1="205.74" x2="-106.68" y2="205.74" width="0.1524" layer="91"/>
 <pinref part="U$4" gate="G$1" pin="G"/>
+<pinref part="C10" gate="G$1" pin="1"/>
+<wire x1="-124.46" y1="205.74" x2="-124.46" y2="210.82" width="0.1524" layer="91"/>
+<junction x="-124.46" y="210.82"/>
 </segment>
 </net>
@@
 <pinref part="R2" gate="G$1" pin="2"/>
 <wire x1="-111.76" y1="-30.48" x2="-128.27" y2="-30.48" width="0.1524" layer="91"/>
+<wire x1="-127" y1="-35.56" x2="-116.84" y2="-35.56" width="0.1524" layer="91"/>
 <wire x1="-116.84" y1="-35.56" x2="-111.76" y2="-35.56" width="0.1524" layer="91"/>
 <wire x1="-111.76" y1="-35.56" x2="-106.68" y2="-35.56" width="0.1524" layer="91"/>
@@
 <wire x1="-106.68" y1="-40.64" x2="-96.52" y2="-40.64" width="0.1524" layer="91"/>
 <pinref part="U$5" gate="G$1" pin="G"/>
+<pinref part="C13" gate="G$1" pin="1"/>
+<wire x1="-116.84" y1="-40.64" x2="-116.84" y2="-35.56" width="0.1524" layer="91"/>
+<junction x="-116.84" y="-35.56"/>
 </segment>
 </net>
@@
 <pinref part="R13" gate="G$1" pin="2"/>
 <wire x1="299.72" y1="-35.56" x2="283.21" y2="-35.56" width="0.1524" layer="91"/>
+<wire x1="287.02" y1="-40.64" x2="294.64" y2="-40.64" width="0.1524" layer="91"/>
 <wire x1="294.64" y1="-40.64" x2="299.72" y2="-40.64" width="0.1524" layer="91"/>
 <wire x1="299.72" y1="-40.64" x2="304.8" y2="-40.64" width="0.1524" layer="91"/>
@@
 <wire x1="304.8" y1="-45.72" x2="312.42" y2="-45.72" width="0.1524" layer="91"/>
 <pinref part="U$7" gate="G$1" pin="G"/>
-</segment>
-</net>
+<pinref part="C17" gate="G$1" pin="1"/>
+<wire x1="294.64" y1="-45.72" x2="294.64" y2="-40.64" width="0.1524" layer="91"/>
+<junction x="294.64" y="-40.64"/>
+</segment>
+</net>
+<net name="FILTEREDNE" class="2">
+<segment>
+<pinref part="C15" gate="G$1" pin="1"/>
+<wire x1="307.34" y1="210.82" x2="302.26" y2="210.82" width="0.1524" layer="91"/>
+<label x="295.91" y="220.98" size="1.778" layer="95" rot="R180" xref="yes"/>
+<pinref part="R6" gate="G$1" pin="2"/>
+<wire x1="312.42" y1="220.98" x2="295.91" y2="220.98" width="0.1524" layer="91"/>
+<wire x1="297.18" y1="215.9" x2="302.26" y2="215.9" width="0.1524" layer="91"/>
+<wire x1="302.26" y1="215.9" x2="312.42" y2="215.9" width="0.1524" layer="91"/>
+<wire x1="312.42" y1="215.9" x2="317.5" y2="215.9" width="0.1524" layer="91"/>
+<wire x1="317.5" y1="215.9" x2="317.5" y2="210.82" width="0.1524" layer="91"/>
+<wire x1="312.42" y1="208.28" x2="312.42" y2="215.9" width="0.1524" layer="91"/>
+<junction x="312.42" y="215.9"/>
+<wire x1="312.42" y1="220.98" x2="312.42" y2="215.9" width="0.1524" layer="91"/>
+<pinref part="R12" gate="G$1" pin="2"/>
+<wire x1="312.42" y1="208.28" x2="317.5" y2="208.28" width="0.1524" layer="91"/>
+<wire x1="317.5" y1="210.82" x2="325.12" y2="210.82" width="0.1524" layer="91"/>
+<pinref part="U$8" gate="G$1" pin="G"/>
+<wire x1="302.26" y1="210.82" x2="302.26" y2="215.9" width="0.1524" layer="91"/>
+<junction x="302.26" y="215.9"/>
+</segment>
+</net>

Commit message: made changes to board, almost done.
Parts:
- U$10, U$11, U$12, U$13: device LEDs:RED_LED -> LEDs_new:RED_LED
Changed lines of the file:
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@@
 <part name="GND22" library="quadparts_prebuilt" deviceset="BAT_GND" device=""/>
 <part name="P+12" library="quadparts_brandon" deviceset="3V" device=""/>
-<part name="U$10" library="LEDs" deviceset="RED_LED" device="" value="RED"/>
+<part name="U$10" library="LEDs_new" deviceset="RED_LED" device="" value="RED"/>
 <part name="GND23" library="quadparts_prebuilt" deviceset="GND" device=""/>
 <part name="R1" library="quadparts_prebuilt" deviceset="RESISTOR_" device="SMD-2012-0805" value="330"/>
-<part name="U$11" library="LEDs" deviceset="RED_LED" device="" value="RED"/>
+<part name="U$11" library="LEDs_new" deviceset="RED_LED" device="" value="RED"/>
 <part name="GND24" library="quadparts_prebuilt" deviceset="GND" device=""/>
 <part name="R7" library="quadparts_prebuilt" deviceset="RESISTOR_" device="SMD-2012-0805" value="330"/>
-<part name="U$12" library="LEDs" deviceset="RED_LED" device="" value="RED"/>
+<part name="U$12" library="LEDs_new" deviceset="RED_LED" device="" value="RED"/>
 <part name="GND26" library="quadparts_prebuilt" deviceset="GND" device=""/>
 <part name="R8" library="quadparts_prebuilt" deviceset="RESISTOR_" device="SMD-2012-0805" value="330"/>
-<part name="U$13" library="LEDs" deviceset="RED_LED" device="" value="RED"/>
+<part name="U$13" library="LEDs_new" deviceset="RED_LED" device="" value="RED"/>
 <part name="GND28" library="quadparts_prebuilt" deviceset="GND" device=""/>
 <part name="R15" library="quadparts_prebuilt" deviceset="RESISTOR_" device="SMD-2012-0805" value="330"/>
@@
 <instance part="GND1" gate="1" x="10.16" y="27.94"/>
 <instance part="GND2" gate="1" x="20.32" y="27.94"/>
-<instance part="GND3" gate="1" x="91.44" y="2.54"/>
+<instance part="GND3" gate="1" x="91.44" y="5.08"/>
 <instance part="GND6" gate="1" x="106.68" y="38.1"/>
 <instance part="GND7" gate="1" x="116.84" y="38.1"/>
@@
 </busses>
 <nets>
-<net name="GND" class="2">
+<net name="GND" class="0">
 <segment>
 <pinref part="JPADDED" gate="G$1" pin="6"/>
@@
 </segment>
 <segment>
-<wire x1="91.44" y1="17.78" x2="91.44" y2="5.08" width="0.1524" layer="91"/>
+<wire x1="91.44" y1="17.78" x2="91.44" y2="7.62" width="0.1524" layer="91"/>
 <wire x1="88.9" y1="17.78" x2="91.44" y2="17.78" width="0.1524" layer="91"/>
 <wire x1="88.9" y1="20.32" x2="91.44" y2="20.32" width="0.1524" layer="91"/>
