File: quadcopter.sch (EAGLE design)
At the start: 73 parts, among them J1 AVR_SPI_PRG_6NS, U3 ATMEGA128RFA1

Commit message: almost done with board, have 3 airwires
Connections:
- net BAT_GND: now also BATT1.N, U$1.P$1; no longer U$1.P$2
- net GND: now also U$1.P$2; no longer BATT1.N, U$1.P$1
Changed lines of the file:
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@@
 <instance part="U$6" gate="G$1" x="314.96" y="238.76"/>
 <instance part="U$9" gate="G$1" x="302.26" y="-17.78"/>
-<instance part="GND25" gate="1" x="-45.72" y="111.76"/>
-<instance part="GND30" gate="1" x="-88.9" y="114.3"/>
+<instance part="GND25" gate="1" x="-86.36" y="114.3"/>
+<instance part="GND30" gate="1" x="-45.72" y="114.3"/>
 <instance part="C3" gate="G$1" x="-38.1" y="116.84"/>
 <instance part="GND42" gate="1" x="-33.02" y="106.68"/>
@@
 </segment>
 <segment>
-<pinref part="U$1" gate="G$1" pin="P$1"/>
-<pinref part="GND30" gate="1" pin="GND"/>
-<wire x1="-81.28" y1="119.38" x2="-88.9" y2="119.38" width="0.1524" layer="91"/>
-<pinref part="BATT1" gate="G$1" pin="N"/>
-<wire x1="-88.9" y1="119.38" x2="-88.9" y2="116.84" width="0.1524" layer="91"/>
-<wire x1="-91.44" y1="127" x2="-91.44" y2="119.38" width="0.1524" layer="91"/>
-<wire x1="-91.44" y1="119.38" x2="-88.9" y2="119.38" width="0.1524" layer="91"/>
-<junction x="-88.9" y="119.38"/>
-</segment>
-<segment>
 <wire x1="144.78" y1="73.66" x2="144.78" y2="58.42" width="0.1524" layer="91"/>
 <pinref part="B1" gate="G$1" pin="GND@5"/>
@@
 <pinref part="C8" gate="G$1" pin="1"/>
 <pinref part="GND39" gate="1" pin="GND"/>
+</segment>
+<segment>
+<pinref part="U$1" gate="G$1" pin="P$2"/>
+<wire x1="-50.8" y1="119.38" x2="-45.72" y2="119.38" width="0.1524" layer="91"/>
+<pinref part="GND30" gate="1" pin="GND"/>
+<wire x1="-45.72" y1="116.84" x2="-45.72" y2="119.38" width="0.1524" layer="91"/>
 </segment>
 </net>
@@
 </segment>
 </net>
-<net name="BAT_GND" class="0">
-<segment>
-<pinref part="U$1" gate="G$1" pin="P$2"/>
-<pinref part="GND25" gate="1" pin="BAT_GND"/>
-<wire x1="-50.8" y1="119.38" x2="-45.72" y2="119.38" width="0.1524" layer="91"/>
-<wire x1="-45.72" y1="119.38" x2="-45.72" y2="114.3" width="0.1524" layer="91"/>
-</segment>
+<net name="BAT_GND" class="2">
 <segment>
 <pinref part="J3" gate="G$1" pin="BAT_GND"/>
@@
 <wire x1="-78.74" y1="-53.34" x2="-78.74" y2="-58.42" width="0.1524" layer="91"/>
 <pinref part="GND47" gate="1" pin="BAT_GND"/>
+</segment>
+<segment>
+<pinref part="U$1" gate="G$1" pin="P$1"/>
+<wire x1="-81.28" y1="119.38" x2="-86.36" y2="119.38" width="0.1524" layer="91"/>
+<pinref part="BATT1" gate="G$1" pin="N"/>
+<wire x1="-86.36" y1="119.38" x2="-91.44" y2="119.38" width="0.1524" layer="91"/>
+<wire x1="-91.44" y1="127" x2="-91.44" y2="119.38" width="0.1524" layer="91"/>
+<pinref part="GND25" gate="1" pin="BAT_GND"/>
+<wire x1="-86.36" y1="116.84" x2="-86.36" y2="119.38" width="0.1524" layer="91"/>
+<junction x="-86.36" y="119.38"/>
 </segment>
 </net>
@@
 </segment>
 </net>
-<net name="N$6" class="0">
+<net name="N$6" class="2">
 <segment>
 <pinref part="BATT1" gate="G$1" pin="P"/>

Commit message: fixed crystal routing and antenna routing, moved motor recouping caps, and replaced wrong filter diodes
Parts:
- D1, D2, D3, D4: value 20V-500MA -> 360mV; device quadparts_prebuilt:DIODE-LED_SMD-2012-0805 -> quadparts_prebuilt:DIODE-SCHOTTKY_SMD-SOD123-360MV
Changed lines of the file:
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@@
 <part name="GND16" library="quadparts_prebuilt" deviceset="GND" device=""/>
 <part name="GND17" library="quadparts_prebuilt" deviceset="GND" device=""/>
-<part name="D2" library="quadparts_prebuilt" deviceset="DIODE-LED_" device="SMD-2012-0805" value="20V-500MA"/>
+<part name="D2" library="quadparts_prebuilt" deviceset="DIODE-SCHOTTKY_" device="SMD-SOD123-360MV" value="360mV"/>
 <part name="C6" library="quadparts_prebuilt" deviceset="CAPACITOR-POL_" device="SMD-7043-D_TANTALUM-220UF" value="100uF"/>
 <part name="C10" library="quadparts_prebuilt" deviceset="CAPACITOR-NP_" device="SMD-2012-0805_CERAMIC-1UF" value="0.1uF"/>
 <part name="R3" library="quadparts_prebuilt" deviceset="RESISTOR_" device="SMD-2012-0805-100" value="100"/>
 <part name="R4" library="quadparts_prebuilt" deviceset="RESISTOR_" device="SMD-2012-0805-10K" value="10K"/>
-<part name="D1" library="quadparts_prebuilt" deviceset="DIODE-LED_" device="SMD-2012-0805" value="20V-500MA"/>
+<part name="D1" library="quadparts_prebuilt" deviceset="DIODE-SCHOTTKY_" device="SMD-SOD123-360MV" value="360mV"/>
 <part name="C11" library="quadparts_prebuilt" deviceset="CAPACITOR-POL_" device="SMD-7043-D_TANTALUM-220UF" value="100uF"/>
 <part name="C13" library="quadparts_prebuilt" deviceset="CAPACITOR-NP_" device="SMD-2012-0805_CERAMIC-1UF" value="0.1uF"/>
@@
 <part name="R5" library="quadparts_prebuilt" deviceset="RESISTOR_" device="SMD-2012-0805-10K" value="10K"/>
 <part name="GND29" library="quadparts_prebuilt" deviceset="GND" device=""/>
-<part name="D3" library="quadparts_prebuilt" deviceset="DIODE-LED_" device="SMD-2012-0805" value="20V-500MA"/>
+<part name="D3" library="quadparts_prebuilt" deviceset="DIODE-SCHOTTKY_" device="SMD-SOD123-360MV" value="360mV"/>
 <part name="C14" library="quadparts_prebuilt" deviceset="CAPACITOR-POL_" device="SMD-7043-D_TANTALUM-220UF" value="100uF"/>
 <part name="C15" library="quadparts_prebuilt" deviceset="CAPACITOR-NP_" device="SMD-2012-0805_CERAMIC-1UF" value="0.1uF"/>
@@
 <part name="R12" library="quadparts_prebuilt" deviceset="RESISTOR_" device="SMD-2012-0805-10K" value="10K"/>
 <part name="GND33" library="quadparts_prebuilt" deviceset="GND" device=""/>
-<part name="D4" library="quadparts_prebuilt" deviceset="DIODE-LED_" device="SMD-2012-0805" value="20V-500MA"/>
+<part name="D4" library="quadparts_prebuilt" deviceset="DIODE-SCHOTTKY_" device="SMD-SOD123-360MV" value="360mV"/>
 <part name="C16" library="quadparts_prebuilt" deviceset="CAPACITOR-POL_" device="SMD-7043-D_TANTALUM-220UF" value="100uF"/>
 <part name="C17" library="quadparts_prebuilt" deviceset="CAPACITOR-NP_" device="SMD-2012-0805_CERAMIC-1UF" value="0.1uF"/>
@@
 <pinref part="D2" gate="G$1" pin="C"/>
 <wire x1="-106.68" y1="241.3" x2="-101.6" y2="241.3" width="0.1524" layer="91"/>
-<wire x1="-101.6" y1="241.3" x2="-101.6" y2="238.76" width="0.1524" layer="91"/>
+<wire x1="-101.6" y1="241.3" x2="-101.6" y2="236.22" width="0.1524" layer="91"/>
 <wire x1="-124.46" y1="246.38" x2="-124.46" y2="248.92" width="0.1524" layer="91"/>
 <junction x="-124.46" y="246.38"/>
@@
 <pinref part="D1" gate="G$1" pin="C"/>
 <wire x1="-99.06" y1="-5.08" x2="-93.98" y2="-5.08" width="0.1524" layer="91"/>
-<wire x1="-93.98" y1="-5.08" x2="-93.98" y2="-7.62" width="0.1524" layer="91"/>
+<wire x1="-93.98" y1="-5.08" x2="-93.98" y2="-10.16" width="0.1524" layer="91"/>
 <wire x1="-116.84" y1="0" x2="-116.84" y2="2.54" width="0.1524" layer="91"/>
 <junction x="-116.84" y="0"/>
@@
 <pinref part="D4" gate="G$1" pin="C"/>
 <wire x1="312.42" y1="-10.16" x2="317.5" y2="-10.16" width="0.1524" layer="91"/>
-<wire x1="317.5" y1="-10.16" x2="317.5" y2="-12.7" width="0.1524" layer="91"/>
+<wire x1="317.5" y1="-10.16" x2="317.5" y2="-15.24" width="0.1524" layer="91"/>
 <wire x1="294.64" y1="-5.08" x2="294.64" y2="-2.54" width="0.1524" layer="91"/>
 <junction x="294.64" y="-5.08"/>
@@
 <pinref part="D3" gate="G$1" pin="C"/>
 <wire x1="325.12" y1="246.38" x2="330.2" y2="246.38" width="0.1524" layer="91"/>
-<wire x1="330.2" y1="246.38" x2="330.2" y2="243.84" width="0.1524" layer="91"/>
+<wire x1="330.2" y1="246.38" x2="330.2" y2="241.3" width="0.1524" layer="91"/>
 <wire x1="307.34" y1="251.46" x2="307.34" y2="254" width="0.1524" layer="91"/>
 <junction x="307.34" y="251.46"/>
@@
 <wire x1="322.58" y1="238.76" x2="325.12" y2="238.76" width="0.1524" layer="91"/>
 <pinref part="D3" gate="G$1" pin="A"/>
-<wire x1="330.2" y1="233.68" x2="330.2" y2="236.22" width="0.1524" layer="91"/>
 <wire x1="325.12" y1="238.76" x2="325.12" y2="233.68" width="0.1524" layer="91"/>
 <wire x1="325.12" y1="233.68" x2="330.2" y2="233.68" width="0.1524" layer="91"/>
@@
 <wire x1="-109.22" y1="219.71" x2="-109.22" y2="233.68" width="0.1524" layer="91"/>
 <pinref part="D2" gate="G$1" pin="A"/>
-<wire x1="-101.6" y1="228.6" x2="-101.6" y2="231.14" width="0.1524" layer="91"/>
 <wire x1="-106.68" y1="233.68" x2="-106.68" y2="228.6" width="0.1524" layer="91"/>
 <wire x1="-106.68" y1="228.6" x2="-101.6" y2="228.6" width="0.1524" layer="91"/>
@@
 <wire x1="-99.06" y1="-12.7" x2="-99.06" y2="-17.78" width="0.1524" layer="91"/>
 <wire x1="-99.06" y1="-17.78" x2="-93.98" y2="-17.78" width="0.1524" layer="91"/>
-<wire x1="-93.98" y1="-17.78" x2="-93.98" y2="-15.24" width="0.1524" layer="91"/>
 <wire x1="-101.6" y1="-12.7" x2="-99.06" y2="-12.7" width="0.1524" layer="91"/>
 <pinref part="U$5" gate="G$1" pin="D"/>
@@
 <wire x1="309.88" y1="-17.78" x2="312.42" y2="-17.78" width="0.1524" layer="91"/>
 <pinref part="D4" gate="G$1" pin="A"/>
-<wire x1="317.5" y1="-22.86" x2="317.5" y2="-20.32" width="0.1524" layer="91"/>
 <wire x1="312.42" y1="-17.78" x2="312.42" y2="-22.86" width="0.1524" layer="91"/>
 <wire x1="312.42" y1="-22.86" x2="317.5" y2="-22.86" width="0.1524" layer="91"/>
